File: Eagle Files/Arduino Nano RGB Led Controller.brd (EAGLE design)
At the start: 38.7 x 50.5 mm, 17 parts, among them J1 12V, M1 ARDUINO-NANO-3.0#ISP

Commit message: Logo added at pcb file
My Logo added at pcb file
Parts:
- R1: device pot:3RP/1610N -> rcl:M1206
- R4: device rcl:M1206 -> pot:3RP/1610N
- moved R1 25.1 mm to (21.6, 21.6), turned to 180 degrees
- moved R4 25.1 mm to (3.81, 39.4), turned to 270 degrees
Connections:
- net +5V: now also R4.3; no longer R1.3
- net GND: now also R1.2, R4.1; no longer R1.1, R4.2
- net N$1: now also R4.2; no longer R1.2
- net RED: now also R1.1; no longer R4.1
