File: Eagle Files/Arduino Nano RGB Led Controller.brd (EAGLE design)
At the start: 38.7 x 50.5 mm, 17 parts, among them J1 12V, M1 ARDUINO-NANO-3.0#ISP

Commit message: update
Parts:
- removed J1: 12V, con-jack:DCJ0303
- added D2: 1N4004, diode:DO41-10
- added J2: V-IN 12V 1.5A MAX, con-jack:SPC4078
- moved R1 7.62 mm to (21.6, 14.0)
- moved R2 7.62 mm to (21.6, 21.6), turned to 0 degrees
- moved RED 1.27 mm to (33.0, 20.3)
- turned R3 to 0 degrees
Connections:
- new net N$3: D2.A, J2.3
- net GND: now also J2.1, J2.2; no longer J1.1, J1.2
- net VIN: now also D2.C; no longer J1.3
Routing:
- net RED: track 65.3 -> 36.4 mm
- net +5V: track 97.9 -> 69.2 mm
- net SDA: track 33.2 -> 20.5 mm, vias 2 -> 0
- net VIN: track 45.4 -> 33.3 mm, vias 1 -> 0
- net D9: track 38.7 -> 26.9 mm, vias 0 -> 1
- net SCL: track 26.5 -> 16.3 mm, vias 2 -> 1
- net BLUE: track 76.8 -> 68.9 mm
- net N$3: track 0.00 -> 5.20 mm
- net D10: track 27.8 -> 23.8 mm
- net D2: track 35.4 -> 31.5 mm, vias 0 -> 1
- net +3V3: track 42.3 -> 38.4 mm
- net N$1: track 28.3 -> 31.6 mm
- net D11: track 23.0 -> 24.5 mm
- net D3: track 22.6 -> 22.8 mm, vias 0 -> 1
Other:
- board text added: "D2 = 12V - 1.5A"
- board text added: "R1,2,3,4,5,6 = 10K R7 = 330R"
- board text added: "RED GREEN BLUE = IRFZ44N"
- board text added: "VILIAS 2016"
- board text removed: "VILIAS ©2016"
