File: Eagle Files/Standalone/RGB Led Controller.sch (EAGLE design)
At the start: 26 parts, among them IC1 7805TV, U1 ATMEGA328P_PDIP, X1 Max 12V in

Commit message: update stand alone
Parts:
- added D1: 1N4004, diode:1N4004
Connections:
- new net N$11: D1.A, X1-1.KL
- net +12V: now also D1.C; no longer X1-1.KL
Changed lines of the file:
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@@
 <part name="H7" library="holes" deviceset="MOUNT-PAD-ROUND" device="3.0"/>
 <part name="H8" library="holes" deviceset="MOUNT-PAD-ROUND" device="3.0"/>
+<part name="D1" library="diode" deviceset="1N4004" device=""/>
 </parts>
 <sheets>
@@
 <instance part="H7" gate="G$1" x="58.42" y="15.24" rot="R90"/>
 <instance part="H8" gate="G$1" x="66.04" y="15.24" rot="R90"/>
+<instance part="D1" gate="1" x="12.7" y="73.66"/>
 </instances>
 <busses>
@@
 <segment>
 <pinref part="IC1" gate="A1" pin="VI"/>
-<pinref part="X1" gate="-1" pin="KL"/>
 <wire x1="38.1" y1="73.66" x2="22.86" y2="73.66" width="0.1524" layer="91"/>
 <pinref part="SUPPLY1" gate="+12V" pin="+12V"/>
-<wire x1="22.86" y1="73.66" x2="5.08" y2="73.66" width="0.1524" layer="91"/>
 <wire x1="22.86" y1="83.82" x2="22.86" y2="73.66" width="0.1524" layer="91"/>
 <pinref part="C1" gate="G$1" pin="+"/>
 <wire x1="22.86" y1="63.5" x2="22.86" y2="73.66" width="0.1524" layer="91"/>
 <junction x="22.86" y="73.66"/>
+<wire x1="15.24" y1="73.66" x2="22.86" y2="73.66" width="0.1524" layer="91"/>
+<pinref part="D1" gate="1" pin="C"/>
 </segment>
 <segment>
@@
 </segment>
 </net>
+<net name="N$11" class="1">
+<segment>
+<pinref part="X1" gate="-1" pin="KL"/>
+<pinref part="D1" gate="1" pin="A"/>
+<wire x1="5.08" y1="73.66" x2="10.16" y2="73.66" width="0.1524" layer="91"/>
+</segment>
+</net>
